File: Hardware/Schematic - Ebook Reader vFinal v37.sch (EAGLE design)
At the start: 103 parts, among them IC1 BD5229G-TR, IC4 XC6220A331MR-G, J1 FH34SRJ-24S-0.5SH_99_, J2 SAMACSYS_PARTS_USB4110-GF-A, J3 QWIIC_RIGHT_ANGLE, J4 112A-TAAR-R03_ATTEND, Q1 20V/4.2A/52mΩ/1.4W, Q2 20V/4.2A/52mΩ/1.4W, Q3 SI1308EDL-T1-GE3, U1 W25Q512JVEIQ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

Commit message: Hardware updated
Parts:
- renumbered TP1 to TX, TP10 to EPD_CS, TP11 to EPD_DC, TP12 to EPD_RST, TP13 to EPD_3V3_C, TP14 to VBUS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
Connections:
- net GND: now also EPD_C8.1
Other:
- moved on the sheet: EPD_C8
