File: Hardware/Schematic_-_Ebook_Reader_vFinal_v58.brd (EAGLE design)
At the start: 170.2 x 111.4 mm, 103 parts, among them IC1 BD5229G-TR, IC4 XC6220A331MR-G, J1 FH34SRJ-24S-0.5SH_99_, J2 SAMACSYS_PARTS_USB4110-GF-A, J3 QWIIC_RIGHT_ANGLE, J4 112A-TAAR-R03_ATTEND, Q1 20V/4.2A/52mΩ/1.4W, Q2 20V/4.2A/52mΩ/1.4W, Q3 SI1308EDL-T1-GE3, U1 W25Q512JVEIQ, U2 ESP32-C6-WROOM-1-N8, U3 DS3231SN#, U4 MAX17048G+T10

Commit message: Hardware updated
Parts:
- renumbered TP1 to TX, TP10 to EPD_CS, TP11 to EPD_DC, TP12 to EPD_RST, TP13 to EPD_3V3_C, TP14 to VBUS, TP15 to INT_RTC, TP16 to 3V3, TP17 to EDP_3V3, TP2 to RX, TP3 to VBAT, TP4 to GND, TP6 to MISO, TP7 to MOSI, TP8 to SCK1, TP9 to EPD_BUSY
Routing:
- net I2C_PW: track 187.2 -> 254.2 mm, vias 5 -> 8
- net GND: track 768.4 -> 734.4 mm
- net SCL: track 220.8 -> 231.6 mm, vias 4 -> 5
- net 3V3: track 516.9 -> 518.0 mm
- net MOSI: track 226.1 -> 227.2 mm
- net EPD_RST: track 159.3 -> 160.3 mm
